Commit message: refactor: moved launch file to commons and the rest to simulation

File: ROS/src/ambition_simulation/urdf/robot.urdf (robot description, URDF)
Before this commit: robot ambition, 21 links, 20 joints
Links:
- link buda: geometry collision mesh filename=package://ambition_simulation/urdf/assets/buda.stl; visual mesh filename=package://ambition_simulation/urdf/assets/buda.stl
- link kolo: geometry collision mesh filename=package://ambition_simulation/urdf/assets/kolo.stl; visual mesh filename=package://ambition_simulation/urdf/assets/kolo.stl
- link kolo_2: geometry collision mesh filename=package://ambition_simulation/urdf/assets/kolo.stl; visual mesh filename=package://ambition_simulation/urdf/assets/kolo.stl
- link kolo_3: geometry collision mesh filename=package://ambition_simulation/urdf/assets/kolo.stl; visual mesh filename=package://ambition_simulation/urdf/assets/kolo.stl
- link kolo_4: geometry collision mesh filename=package://ambition_simulation/urdf/assets/kolo.stl; visual mesh filename=package://ambition_simulation/urdf/assets/kolo.stl
- link pivot: geometry collision mesh filename=package://ambition_simulation/urdf/assets/pivot.stl; visual mesh filename=package://ambition_simulation/urdf/assets/pivot.stl
- link pivot_2: geometry collision mesh filename=package://ambition_simulation/urdf/assets/pivot.stl; visual mesh filename=package://ambition_simulation/urdf/assets/pivot.stl
- link pivot_3: geometry collision mesh filename=package://ambition_simulation/urdf/assets/pivot.stl; visual mesh filename=package://ambition_simulation/urdf/assets/pivot.stl
- link ramie: geometry collision mesh filename=package://ambition_simulation/urdf/assets/ramie.stl; visual mesh filename=package://ambition_simulation/urdf/assets/ramie.stl
- link ramie_2: geometry collision mesh filename=package://ambition_simulation/urdf/assets/ramie.stl; visual mesh filename=package://ambition_simulation/urdf/assets/ramie.stl
- link rod: geometry collision mesh filename=package://ambition_simulation/urdf/assets/rod.stl; visual mesh filename=package://ambition_simulation/urdf/assets/rod.stl
- link rod_2: geometry collision mesh filename=package://ambition_simulation/urdf/assets/rod.stl; visual mesh filename=package://ambition_simulation/urdf/assets/rod.stl
